File: lora.sch (KiCad schematic (older format))
At the start: 34 parts, among them IC3 SX1262IMLTRT, IC4 PE4259-63, J3 Conn_Coaxial, J9 RF Shield, Y3 NT2016SA-32M-END4263A

Commit message: Changed all symbols names from IC to U
Parts:
- renumbered IC3 to U, IC4 to U
Changed lines of the file:
@@
 	6800 4400 8200 4400
 $Comp
-L tardigrade-components:SX1262IMLTRT IC3
+L tardigrade-components:SX1262IMLTRT U
 U 1 1 5F806BC9
 P 4650 3250
-F 0 "IC3" V 4700 3350 50  0000 C CNN
+F 0 "U" V 4700 3350 50  0000 C CNN
 F 1 "SX1262IMLTRT" V 4800 3550 50  0000 C CNN
 F 2 "tardigrade-components:QFN50P400X400X100-25N-D" H 5900 3750 50  0001 L CNN
@@
 $EndComp
 $Comp
-L tardigrade-components:PE4259-63 IC4
+L tardigrade-components:PE4259-63 U
 U 1 1 5F80B8FA
 P 7950 3850
-F 0 "IC4" H 8850 4115 50  0000 C CNN
+F 0 "U" H 8850 4115 50  0000 C CNN
 F 1 "PE4259-63" H 8850 4024 50  0000 C CNN
 F 2 "tardigrade-components:SOT65P210X110-6N" H 9300 3950 50  0001 L CNN

Commit message: Unnecessary note removed
Parts:
- renumbered U to U7, U to U8
Changed lines of the file:
@@
 	6800 4400 8200 4400
 $Comp
-L tardigrade-components:SX1262IMLTRT U
+L tardigrade-components:SX1262IMLTRT U7
 U 1 1 5F806BC9
 P 4650 3250
-F 0 "U" V 4700 3350 50  0000 C CNN
+F 0 "U7" V 4700 3350 50  0000 C CNN
 F 1 "SX1262IMLTRT" V 4800 3550 50  0000 C CNN
 F 2 "tardigrade-components:QFN50P400X400X100-25N-D" H 5900 3750 50  0001 L CNN
@@
 $EndComp
 $Comp
-L tardigrade-components:PE4259-63 U
+L tardigrade-components:PE4259-63 U8
 U 1 1 5F80B8FA
 P 7950 3850
-F 0 "U" H 8850 4115 50  0000 C CNN
+F 0 "U8" H 8850 4115 50  0000 C CNN
 F 1 "PE4259-63" H 8850 4024 50  0000 C CNN
 F 2 "tardigrade-components:SOT65P210X110-6N" H 9300 3950 50  0001 L CNN

Commit message: Added footprint assignment
Parts:
- L4: footprint Inductor_SMD:L_0402_1005Metric -> Inductor_SMD:L_0805_2012Metric
Changed lines of the file:
@@
 F 0 "L4" V 3150 3800 50  0000 C CNN
 F 1 "15uH" V 3050 3650 50  0000 C CNN
-F 2 "Inductor_SMD:L_0402_1005Metric" H 3100 3650 50  0001 C CNN
+F 2 "Inductor_SMD:L_0805_2012Metric" H 3100 3650 50  0001 C CNN
 F 3 "~" H 3100 3650 50  0001 C CNN
 	1    3100 3650

Commit message: Major change of the layout (reviewed) for V1.1
Parts:
- renumbered C27 to C29, C28 to C30, C29 to C31, C30 to C32, C31 to C33, C32 to C34, C33 to C35, C34 to C36, C35 to C37, C36 to C38, C37 to C39, C38 to C40, C39 to C41, C40 to C42, C41 to C43, C42 to C44, C43 to C45, C44 to C46, J9 to J3, J3 to J4, R21 to R18, R22 to R19, R23 to R20, U7 to U4, U8 to U5
