File: mcu.sch (KiCad schematic (older format))
At the start: 23 parts, among them U6 LPC55S16JBD64E, Y1 16 MHz, Y2 32.768 kHz

Commit message: Added footprint assignment
Parts:
- C22, C26: footprint Capacitor_SMD:C_0402_1005Metric -> Capacitor_SMD:C_0603_1608Metric
- L3: footprint Inductor_SMD:L_0402_1005Metric -> Inductor_SMD:L_0805_2012Metric
Changed lines of the file:
@@
 F 0 "C26" H 7050 4750 50  0000 L CNN
 F 1 "22uF" H 7050 4550 50  0000 L CNN
-F 2 "Capacitor_SMD:C_0402_1005Metric" H 7088 4500 50  0001 C CNN
+F 2 "Capacitor_SMD:C_0603_1608Metric" H 7088 4500 50  0001 C CNN
 F 3 "~" H 7050 4650 50  0001 C CNN
 	1    7050 4650
@@
 F 0 "C22" H 5300 6050 50  0000 L CNN
 F 1 "22uF" H 5250 5850 50  0000 L CNN
-F 2 "Capacitor_SMD:C_0402_1005Metric" H 5488 5800 50  0001 C CNN
+F 2 "Capacitor_SMD:C_0603_1608Metric" H 5488 5800 50  0001 C CNN
 F 3 "~" H 5450 5950 50  0001 C CNN
 	1    5450 5950
@@
 F 0 "L3" H 5656 5554 50  0000 R CNN
 F 1 "4.7uH" H 5656 5645 50  0000 R CNN
-F 2 "Inductor_SMD:L_0402_1005Metric" H 5700 5600 50  0001 C CNN
+F 2 "Inductor_SMD:L_0805_2012Metric" H 5700 5600 50  0001 C CNN
 F 3 "~" H 5700 5600 50  0001 C CNN
 	1    5700 5600

Commit message: Major change of the layout (reviewed) for V1.1
Parts:
- renumbered C10 to C12, C11 to C13, C12 to C14, C13 to C15, C14 to C16, C15 to C17, C16 to C18, C17 to C19, C18 to C20, C19 to C21, C20 to C22, C21 to C23, C22 to C24, C23 to C25, C24 to C26, C25 to C27, C26 to C28, R18 to R16, R19 to R17, U6 to U8
Connections:
- net SX1262_BUSY: now also U8.4 (PIO1_0/_ADC0_11); no longer U8.3 (PIO0_17)
- net SX1262_NRESET: now also U8.3 (PIO0_17); no longer U8.4 (PIO1_0/_ADC0_11)
- net VSTOR_MEASURE renamed MCU_PIO0_23
